Commit message: Added gmapping code, needs tuning

File: src/shipbot_description/urdf/shipbot.gazebo.xacro (robot description, xacro)
@@ -1,6 +1,6 @@
 <?xml version="1.0"?>
 <robot name="shipbot" xmlns:xacro="http://ros.org/wiki/xacro">
-  <!-- <xacro:arg name="laser_visual"  default="false"/>
-  <xacro:arg name="camera_visual" default="false"/>
+  <xacro:arg name="laser_visual"  default="true"/>
+  <!-- <xacro:arg name="camera_visual" default="false"/>
   <xacro:arg name="imu_visual"    default="false"/> -->
   <gazebo reference="base_link">
@@ -20,50 +20,13 @@
   </gazebo>
   <gazebo>
-    <plugin name="shipbot_controller" filename="libgazebo_ros_diff_drive.so">
-      <legacyMode>false</legacyMode>
-      <alwaysOn>true</alwaysOn>
+    <plugin name="shipbot_controller" filename="libgazebo_ros_planar_move.so">
       <commandTopic>cmd_vel</commandTopic>
       <odometryTopic>odom</odometryTopic>
       <odometryFrame>odom</odometryFrame>
-      <odometrySource>world</odometrySource>
-      <publishOdomTF>true</publishOdomTF>
+      <odometryRate>20.0</odometryRate>
       <robotBaseFrame>base_footprint</robotBaseFrame>
-      <publishWheelTF>false</publishWheelTF>
-      <publishTf>1</publishTf>
-      <publishWheelJointState>false</publishWheelJointState>
-      <updateRate>10</updateRate>
-      <leftJoint>wheel_front_left_joint</leftJoint>
-      <rightJoint>wheel_front_right_joint</rightJoint>
-      <wheelSeparation>0.1778</wheelSeparation>
-      <wheelDiameter>0.066</wheelDiameter>
-      <wheelAcceleration>0</wheelAcceleration>
-      <wheelTorque>5</wheelTorque>
-      <torque>10</torque>
-      <rosDebugLevel>na</rosDebugLevel>
     </plugin>
   </gazebo>
-  <!-- <gazebo>
-    <plugin name="shipbot_controller" filename="libgazebo_ros_mecanum_drive.so">
-      <commandTopic>cmd_vel</commandTopic>
-      <odometryTopic>odom</odometryTopic>
-      <odometryFrame>odom</odometryFrame>
-      <robotBaseFrame>base_footprint</robotBaseFrame>
-      <LeftRear>wheel_rear_left_joint</LeftRear>
-      <LeftFront>wheel_front_left_joint</LeftFront>
-      <RightFront>wheel_front_right_joint</RightFront>
-      <RightRear>wheel_rear_right_joint</RightRear>
-      <odometryRate>30</odometryRate>
-      <publishWheelTF>true</publishWheelTF>
-      <publishWheelJointState>true</publishWheelJointState>
-      <WheelTorque>1</WheelTorque>
-      <WheelSeparationW>0.1778</WheelSeparationW>
-      <WheelSeparationL>0.1778</WheelSeparationL>
-      <wheelAccel>5</wheelAccel>
-      <wheelDiameter>0.066</wheelDiameter>
-      <publishOdom>true</publishOdom>
-      <isRollerModel>true</isRollerModel>
-    </plugin>
-  </gazebo> -->
-  <!-- <gazebo reference="base_scan">
+  <gazebo reference="base_scan">
     <material>Gazebo/FlatBlack</material>
     <sensor type="ray" name="lds_lfcd_sensor">
@@ -76,6 +39,6 @@
             <samples>360</samples>
             <resolution>1</resolution>
-            <min_angle>0.0</min_angle>
-            <max_angle>6.28319</max_angle>
+            <min_angle>-1.222</min_angle>
+            <max_angle>1.222</max_angle>
           </horizontal>
         </scan>
@@ -96,5 +59,5 @@
       </plugin>
     </sensor>
-  </gazebo> -->
+  </gazebo>
 <!--link : https://www.raspberrypi.org/documentation/hardware/camera/-->
   <!-- <gazebo reference="camera_rgb_frame">

File: src/shipbot_description/urdf/shipbot.urdf.xacro (robot description, xacro)
@@ -34,5 +34,5 @@
     <parent link="base_link"/>
     <child link="wheel_front_left_link"/>
-    <origin xyz="0.0889 0.0889 0.023" rpy="-1.57 0 0"/>
+    <origin xyz="0.0889 0.0889 -0.023" rpy="-1.57 0 0"/>
     <axis xyz="0 0 1"/>
   </joint>
@@ -62,5 +62,5 @@
     <parent link="base_link"/>
     <child link="wheel_front_right_link"/>
-    <origin xyz="0.0889 -0.0889 0.023" rpy="-1.57 0 0"/>
+    <origin xyz="0.0889 -0.0889 -0.023" rpy="-1.57 0 0"/>
     <axis xyz="0 0 1"/>
   </joint>
@@ -90,5 +90,5 @@
     <parent link="base_link"/>
     <child link="wheel_rear_right_link"/>
-    <origin xyz="-0.0889 -0.0889 0.023" rpy="-1.57 0 0"/>
+    <origin xyz="-0.0889 -0.0889 -0.023" rpy="-1.57 0 0"/>
     <axis xyz="0 0 1"/>
   </joint>
@@ -118,5 +118,5 @@
     <parent link="base_link"/>
     <child link="wheel_rear_left_link"/>
-    <origin xyz="-0.0889 0.0889 0.023" rpy="-1.57 0 0"/>
+    <origin xyz="-0.0889 0.0889 -0.023" rpy="-1.57 0 0"/>
     <axis xyz="0 0 1"/>
   </joint>
@@ -149,12 +149,12 @@
   </joint>
   <link name="imu_link"/> -->
-  <!-- <joint name="scan_joint" type="fixed">
+  <joint name="scan_joint" type="fixed">
     <parent link="base_link"/>
     <child link="base_scan"/>
-    <origin xyz="-0.064 0 0" rpy="0 0 0"/>
+    <origin xyz="0.15 0 -0.0158" rpy="0 0 0"/>
   </joint>
   <link name="base_scan">
     <visual>
-      <origin xyz="0.015 0 -0.0065" rpy="0 0 0"/>
+      <origin xyz="0 0 0" rpy="0 0 0"/>
       <geometry>
         <cylinder length="0.0315" radius="0.055"/>
@@ -163,5 +163,5 @@
     </visual>
     <collision>
-      <origin xyz="0.015 0 -0.0065" rpy="0 0 0"/>
+      <origin xyz="0 0 0" rpy="0 0 0"/>
       <geometry>
         <cylinder length="0.0315" radius="0.055"/>
@@ -176,5 +176,5 @@
     </inertial>
   </link>
-  <joint name="camera_joint" type="fixed">
+  <!-- <joint name="camera_joint" type="fixed">
     <origin xyz="0.073 -0.011 0.084" rpy="0 0 0"/>
     <parent link="base_link"/>
